File: Hardware/Ink_Time.brd (EAGLE design)
At the start: 46 x 35 mm, 105 parts, among them IC1 BQ25180YBGR, IC2 DRV2605YZFR, IC3 BMA423, IC9 RT6160AWSC_RT6160AWSC, J1 503480-2400, J2 TC2030-IDC, J4 KH-TYPE-C-16P_KH-TYPE-C-16P, Q1 20V/4.2A/52mΩ/1.4W, Q3 SI1308EDL-T1-GE3, U1 NRF52840_QF, U3 MAX17048G+T10, X1 32MHz, X2 32.768kHz

Commit message: via stitching
Parts:
- moved C23 0.64 mm to (-16.0, 15.0)
- moved C37 0.20 mm to (-7.75, 13.6)
Routing:
- net GND: track 347.9 -> 358.3 mm, vias 5 -> 18
- net VREG: track 18.3 -> 20.4 mm
